Commit message: add(fishbot_description): 添加轮子和转向器的XACRO描述文件，并更新机器人URDF以包含新组件

File: fishbot_description/urdf/fishbot/base.urdf.xacro (robot description, xacro)
@@ -2,4 +2,6 @@
 <robot xmlns:xacro="http://www.ros.org/wiki/xacro">
     <xacro:macro name="base_xacro" params="length radius">
+        <link name="base_footprint">
+        </link>
         <link name="base_link">
             <visual>
@@ -8,9 +10,14 @@
                     <cylinder radius="${radius}" length="${length}"/>
                 </geometry>
-                <material name="Black">
-                    <color rgba="0.0 0.0 0.0 1.0"/>
+                <material name="Gray">
+                    <color rgba="0.7 0.7 0.7 0.5"/>
                 </material>
             </visual>
         </link>
+        <joint name="joint_name" type="fixed">
+            <origin xyz="0.0 0.0 ${length/2.0 + 0.032 - 0.001}" rpy="0.0 0.0 0.0"/>
+            <parent link="base_footprint"/>
+            <child link="base_link"/>
+        </joint>
     </xacro:macro>
 </robot>

File: fishbot_description/urdf/fishbot/fishbot.urdf.xacro (robot description, xacro)
@@ -5,7 +5,13 @@
     <xacro:include filename="$(find fishbot_description)/urdf/fishbot/sensor/camera.urdf.xacro" />
     <xacro:include filename="$(find fishbot_description)/urdf/fishbot/sensor/laser.urdf.xacro" />
+    <xacro:include filename="$(find fishbot_description)/urdf/fishbot/actuator/wheel.urdf.xacro" />
+    <xacro:include filename="$(find fishbot_description)/urdf/fishbot/actuator/caster.urdf.xacro" />
     <xacro:base_xacro length="0.12" radius="0.10" />
-    <xacro:imu_xacro xyz="0.0 0.0 0.07" />
-    <xacro:camera_xacro xyz="0.10 0.0 0.075" />
+    <xacro:imu_xacro xyz="0.0 0.0 0.02" />
+    <xacro:camera_xacro xyz="0.10 0.0 0.07" />
     <xacro:laser_xacro xyz="0.0 0.0 0.11" />
+    <xacro:wheel_xacro name="left_wheel" xyz="0.0 0.10 -0.06" />
+    <xacro:wheel_xacro name="right_wheel" xyz="0.0 -0.10 -0.06" />
+    <xacro:caster_xacro name="front_caster" xyz="0.08 0.0 -0.076" />
+    <xacro:caster_xacro name="back_caster" xyz="-0.08 0.0 -0.076" />
 </robot>
