Commit message: add(fishbot_description): 为各个组件添加碰撞模型，包括轮子、摄像头、IMU和激光传感器

File: fishbot_description/urdf/fishbot/actuator/caster.urdf.xacro (robot description, xacro)
@@ -12,4 +12,13 @@
                 </material>
             </visual>
+            <collision>
+                <origin rpy="0 0 0" xyz="0 0 0"/>
+                <geometry>
+                    <sphere radius="0.016"/>
+                </geometry>
+                <material name="Yellow">
+                    <color rgba="1.0 1.0 0.0 0.8"/>
+                </material>
+            </collision>
         </link>
         <joint name="${name}_wheel_joint" type="fixed">

File: fishbot_description/urdf/fishbot/actuator/wheel.urdf.xacro (robot description, xacro)
@@ -12,4 +12,13 @@
                 </material>
             </visual>
+            <collision>
+                <origin rpy="1.57079 0 0" xyz="0 0 0"/>
+                <geometry>
+                    <cylinder radius="0.032" length="0.04" />
+                </geometry>
+                <material name="Yellow">
+                    <color rgba="1.0 1.0 0.0 0.8"/>
+                </material>
+            </collision>
         </link>
         <joint name="${name}_joint" type="continuous">

File: fishbot_description/urdf/fishbot/base.urdf.xacro (robot description, xacro)
@@ -14,4 +14,13 @@
                 </material>
             </visual>
+            <collision>
+                <origin rpy="0 0 0" xyz="0 0 0"/>
+                <geometry>
+                    <cylinder radius="${radius}" length="${length}"/>
+                </geometry>
+                <material name="Gray">
+                    <color rgba="0.7 0.7 0.7 0.5"/>
+                </material>
+            </collision>
         </link>
         <joint name="joint_name" type="fixed">

File: fishbot_description/urdf/fishbot/sensor/camera.urdf.xacro (robot description, xacro)
@@ -12,4 +12,13 @@
                 </material>
             </visual>
+            <collision>
+                <origin rpy="0 0 0" xyz="0 0 0"/>
+                <geometry>
+                    <box size="0.02 0.10 0.02"/>
+                </geometry>
+                <material name="White">
+                    <color rgba="1.0 1.0 1.0 0.5"/>
+                </material>
+            </collision>
         </link>
         <joint name="camera_joint" type="fixed">

File: fishbot_description/urdf/fishbot/sensor/imu.urdf.xacro (robot description, xacro)
@@ -12,4 +12,13 @@
                 </material>
             </visual>
+            <collision>
+                <origin rpy="0 0 0" xyz="0 0 0"/>
+                <geometry>
+                    <box size="0.02 0.02 0.02"/>
+                </geometry>
+                <material name="White">
+                    <color rgba="1.0 1.0 1.0 0.5"/>
+                </material>
+            </collision>
         </link>
         <joint name="imu_joint" type="fixed">

File: fishbot_description/urdf/fishbot/sensor/laser.urdf.xacro (robot description, xacro)
@@ -12,4 +12,13 @@
                 </material>
             </visual>
+            <collision>
+                <origin rpy="0 0 0" xyz="0 0 0"/>
+                <geometry>
+                    <cylinder radius="0.01" length="0.10"/>
+                </geometry>
+                <material name="White">
+                    <color rgba="1.0 1.0 1.0 1.0"/>
+                </material>
+            </collision>
         </link>
         <link name="laser_link">
@@ -23,4 +32,13 @@
                 </material>
             </visual>
+            <collision>
+                <origin rpy="0 0 0" xyz="0 0 0"/>
+                <geometry>
+                    <cylinder radius="0.02" length="0.02"/>
+                </geometry>
+                <material name="White">
+                    <color rgba="0.0 0.0 0.0 0.5"/>
+                </material>
+            </collision>
         </link>
         <joint name="laser_joint" type="fixed">

Commit message: add(fishbot_description): 为各个组件添加Gazebo仿真配置，包括轮子、转向器、基础、相机、IMU和激光传感器

File: fishbot_description/urdf/fishbot/actuator/caster.urdf.xacro (robot description, xacro)
@@ -29,4 +29,11 @@
             <origin xyz="${xyz}" rpy="0.0 0.0 0.0"/>
         </joint>
+        <gazebo reference="${name}_link">
+            <mu1>0.0</mu1>
+            <mu2>0.0</mu2>
+            <kp>1000000000.0</kp>
+            <kd>1.0</kd>
+            <material>Gazebo/Yellow</material>
+        </gazebo>
     </xacro:macro>
 </robot>

File: fishbot_description/urdf/fishbot/actuator/wheel.urdf.xacro (robot description, xacro)
@@ -30,4 +30,11 @@
             <axis xyz="0 1 0"/>
         </joint>
+        <gazebo reference="${name}_link">
+            <mu1>20.0</mu1>
+            <mu2>20.0</mu2>
+            <kp>1000000000.0</kp>
+            <kd>1.0</kd>
+            <material>Gazebo/Yellow</material>
+        </gazebo>
     </xacro:macro>
 </robot>

File: fishbot_description/urdf/fishbot/base.urdf.xacro (robot description, xacro)
@@ -31,4 +31,9 @@
             <child link="base_link"/>
         </joint>
+        <gazebo reference="base_link">
+            <material>
+                Gazebo/GreyTransparent
+            </material>
+        </gazebo>
     </xacro:macro>
 </robot>

File: fishbot_description/urdf/fishbot/sensor/camera.urdf.xacro (robot description, xacro)
@@ -29,4 +29,9 @@
             <origin xyz="${xyz}" rpy="0.0 0.0 0.0"/>
         </joint>
+        <gazebo reference="imu_link">
+            <material>
+                Gazebo/GreyTransparent
+            </material>
+        </gazebo>
     </xacro:macro>
 </robot>

File: fishbot_description/urdf/fishbot/sensor/imu.urdf.xacro (robot description, xacro)
@@ -29,4 +29,9 @@
             <origin xyz="${xyz}" rpy="0.0 0.0 0.0"/>
         </joint>
+        <gazebo reference="imu_link">
+            <material>
+                Gazebo/GreyTransparent
+            </material>
+        </gazebo>
     </xacro:macro>
 </robot>

File: fishbot_description/urdf/fishbot/sensor/laser.urdf.xacro (robot description, xacro)
@@ -55,4 +55,14 @@
             <origin xyz="${xyz}" rpy="0.0 0.0 0.0"/>
         </joint>
+        <gazebo reference="laser_cylinder_link">
+            <material>
+                Gazebo/GreyTransparent
+            </material>
+        </gazebo>
+        <gazebo reference="laser_link">
+            <material>
+                Gazebo/GreyTransparent
+            </material>
+        </gazebo>
     </xacro:macro>
 </robot>
