Commit message: add(fishbot_description): 添加相机传感器的URDF配置，包括相机链接和关节定义

File: fishbot_description/urdf/fishbot/plugins/gazebo_sensor_plugin.xacro (robot description, xacro)
@@ -110,29 +110,29 @@
             </sensor>
         </gazebo>
+        <gazebo reference="camera_link">
+            <sensor type="depth" name="camera_sensor">
+                <plugin name="depth_camera" filename="libgazebo_ros_camera.so">
+                    <frame_name>camera_optical_link</frame_name>
+                </plugin>
+                <always_on>true</always_on>
+                <update_rate>10</update_rate>
+                <camera name="camera">
+                    <horizontal_fov>1.5009831567</horizontal_fov>
+                    <image>
+                        <width>800</width>
+                        <height>600</height>
+                        <format>R8G8B8</format>
+                    </image>
+                    <distortion>
+                        <k1>0.0</k1>
+                        <k2>0.0</k2>
+                        <k3>0.0</k3>
+                        <p1>0.0</p1>
+                        <p2>0.0</p2>
+                        <center>0.5 0.5</center>
+                    </distortion>
+                </camera>
+            </sensor>
+        </gazebo>
     </xacro:macro>
-    <!-- <gazebo reference="camera_link">
-        <sensor type="depth" name="camera_sensor">
-            <plugin name="depth_camera" filename="libgazebo_ros_camera.so">
-                <frame_name>camera_optical_link</frame_name>
-            </plugin>
-            <always_on>true</always_on>
-            <update_rate>10</update_rate>
-            <camera name="camera">
-                <horizontal_fov>1.5009831567</horizontal_fov>
-                <image>
-                    <width>800</width>
-                    <height>600</height>
-                    <format>R8G8B8</format>
-                </image>
-                <distortion>
-                    <k1>0.0</k1>
-                    <k2>0.0</k2>
-                    <k3>0.0</k3>
-                    <p1>0.0</p1>
-                    <p2>0.0</p2>
-                    <center>0.5 0.5</center>
-                </distortion>
-            </camera>
-        </sensor>
-    </gazebo> -->
 </robot>

File: fishbot_description/urdf/fishbot/sensor/camera.urdf.xacro (robot description, xacro)
@@ -24,4 +24,5 @@
             <xacro:box_inertia m="0.1" w="0.02" h="0.10" d="0.02" />
         </link>
+        <link name="camera_optical_link"></link>
         <joint name="camera_joint" type="fixed">
             <parent link="base_link"/>
@@ -29,5 +30,10 @@
             <origin xyz="${xyz}" rpy="0.0 0.0 0.0"/>
         </joint>
-        <gazebo reference="imu_link">
+        <joint name="camera_optical_joint" type="fixed">
+            <parent link="camera_link"/>
+            <child link="camera_optical_link"/>
+            <origin xyz="0 0 0" rpy="${-pi/2} 0.0 ${-pi/2}"/>
+        </joint>
+        <gazebo reference="camera_link">
             <material>
                 Gazebo/GreyTransparent
